File: emcoder.kicad_sch (KiCad schematic)
At the start: 7 parts, among them U5 PC817, U6 PC817

Commit message: little fix / adding images
Parts:
- renumbered R11 to R1, R12 to R6, R14 to R8, R15 to R9, U5 to U1, U6 to U3, enc1 to enc0
Changed lines of the file:
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@@
 (kicad_sch
-	(version 20231120)
+	(version 20250114)
 	(generator "eeschema")
-	(generator_version "8.0")
+	(generator_version "9.0")
 	(paper "A4")
 	(junction
@@
 		(shape input)
 		(at 99.06 64.77 180)
-		(fields_autoplaced yes)
 		(effects
 			(font
@@
 		(shape input)
 		(at 160.02 82.55 180)
-		(fields_autoplaced yes)
 		(effects
 			(font
@@
 		(shape input)
 		(at 160.02 74.93 180)
-		(fields_autoplaced yes)
 		(effects
 			(font
@@
 		(shape input)
 		(at 138.43 64.77 0)
-		(fields_autoplaced yes)
 		(effects
 			(font
@@
 		(shape input)
 		(at 99.06 81.28 180)
-		(fields_autoplaced yes)
 		(effects
 			(font
@@
 		(dnp no)
 		(fields_autoplaced yes)
-		(property "Reference" "enc1"
+		(property "Reference" "enc0"
 			(at 166.37 77.4699 90)
 			(effects
@@
 		(on_board yes)
 		(dnp no)
-		(property "Reference" "R11"
+		(property "Reference" "R1"
 			(at 105.41 55.88 90)
 			(effects
@@
 		(on_board yes)
 		(dnp no)
-		(property "Reference" "R15"
+		(property "Reference" "R9"
 			(at 129.54 78.74 90)
 			(effects
@@
 		(on_board yes)
 		(dnp no)
-		(property "Reference" "U5"
+		(property "Reference" "U1"
 			(at 118.11 76.2 0)
 			(effects
@@
 		(on_board yes)
 		(dnp no)
-		(property "Reference" "U6"
+		(property "Reference" "U3"
 			(at 118.11 92.71 0)
 			(effects
@@
 		(on_board yes)
 		(dnp no)
-		(property "Reference" "R12"
+		(property "Reference" "R6"
 			(at 105.41 72.39 90)
 			(effects
@@
 		(on_board yes)
 		(dnp no)
-		(property "Reference" "R14"
+		(property "Reference" "R8"
 			(at 129.54 62.23 90)
 			(effects
