File: input.kicad_sch (KiCad schematic)
At the start: 4 parts, among them U48 PC817

Commit message: little fix / adding images
Parts:
- renumbered R110 to R84, R111 to R85, U48 to U35, in3 to ref0
Changed lines of the file:
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@@
 (kicad_sch
-	(version 20231120)
+	(version 20250114)
 	(generator "eeschema")
-	(generator_version "8.0")
+	(generator_version "9.0")
 	(paper "A4")
 	(junction
@@
 		(shape input)
 		(at 106.68 88.9 180)
-		(fields_autoplaced yes)
 		(effects
 			(font
@@
 		(on_board yes)
 		(dnp no)
-		(property "Reference" "R110"
+		(property "Reference" "R84"
 			(at 113.03 80.01 90)
 			(effects
@@
 		(on_board yes)
 		(dnp no)
-		(property "Reference" "R111"
+		(property "Reference" "R85"
 			(at 137.16 86.36 90)
 			(effects
@@
 		(dnp no)
 		(fields_autoplaced yes)
-		(property "Reference" "in3"
+		(property "Reference" "ref0"
 			(at 156.21 90.1699 90)
 			(effects
@@
 		(on_board yes)
 		(dnp no)
-		(property "Reference" "U48"
+		(property "Reference" "U35"
 			(at 125.73 100.33 0)
 			(effects
