File: motor.kicad_sch (KiCad schematic)
At the start: 7 parts, among them U31 PC817, U32 PC817

Commit message: little fix / adding images
Parts:
- renumbered Amp4 to Amp1, R76 to R64, R77 to R65, R78 to R66, R79 to R67, U31 to U25, U32 to U26
Changed lines of the file:
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@@
 (kicad_sch
-	(version 20231120)
+	(version 20250114)
 	(generator "eeschema")
-	(generator_version "8.0")
+	(generator_version "9.0")
 	(paper "A4")
 	(junction
@@
 		(shape input)
 		(at 95.25 110.49 180)
-		(fields_autoplaced yes)
 		(effects
 			(font
@@
 		(shape input)
 		(at 95.25 92.71 180)
-		(fields_autoplaced yes)
 		(effects
 			(font
@@
 		(on_board yes)
 		(dnp no)
-		(property "Reference" "R78"
+		(property "Reference" "R66"
 			(at 124.46 78.74 90)
 			(effects
@@
 		(on_board yes)
 		(dnp no)
-		(property "Reference" "U31"
+		(property "Reference" "U25"
 			(at 111.76 99.06 0)
 			(effects
@@
 		(on_board yes)
 		(dnp no)
-		(property "Reference" "R76"
+		(property "Reference" "R64"
 			(at 100.33 85.09 90)
 			(effects
@@
 		(on_board yes)
 		(dnp no)
-		(property "Reference" "Amp4"
+		(property "Reference" "Amp1"
 			(at 153.67 104.14 0)
 			(effects
@@
 		(on_board yes)
 		(dnp no)
-		(property "Reference" "R77"
+		(property "Reference" "R65"
 			(at 100.33 102.87 90)
 			(effects
@@
 		(on_board yes)
 		(dnp no)
-		(property "Reference" "U32"
+		(property "Reference" "U26"
 			(at 111.76 116.84 0)
 			(effects
@@
 		(on_board yes)
 		(dnp no)
-		(property "Reference" "R79"
+		(property "Reference" "R67"
 			(at 124.46 96.52 90)
 			(effects
