File: output.kicad_sch (KiCad schematic)
At the start: 4 parts, among them U45 PC817

Commit message: little fix / adding images
Parts:
- renumbered R104 to R102, R105 to R103, U45 to U44
Changed lines of the file:
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@@
 (kicad_sch
-	(version 20231120)
+	(version 20250114)
 	(generator "eeschema")
-	(generator_version "8.0")
+	(generator_version "9.0")
 	(paper "A4")
 	(junction
@@
 		(shape input)
 		(at 128.27 92.71 180)
-		(fields_autoplaced yes)
 		(effects
 			(font
@@
 		(on_board yes)
 		(dnp no)
-		(property "Reference" "R104"
+		(property "Reference" "R102"
 			(at 133.35 85.09 90)
 			(effects
@@
 		(on_board yes)
 		(dnp no)
-		(property "Reference" "R105"
+		(property "Reference" "R103"
 			(at 157.48 78.74 90)
 			(effects
@@
 		(on_board yes)
 		(dnp no)
-		(property "Reference" "U45"
+		(property "Reference" "U44"
 			(at 144.78 99.06 0)
 			(effects
