File: rio-motoman.kicad_pcb (KiCad board)
At the start: 2 copper layers, 160 x 100 mm, 183 parts, among them J15 Conn_01x06, J16 Conn_01x06, J2 Conn_02x07_Odd_Even, J4 Conn_01x04, J5 Conn_01x04, U1 PC817, U10 ULN2803A, U11 ULN2803A, U12 MAX485E, U14 PC817, U15 PC817, U17 PC817, U18 PC817, U2 ISO1540, U20 PC817, U21 PC817, U23 PC817, U24 PC817, U25 PC817, U26 PC817, U27 PC817, U28 PC817, U29 PC817, U3 PC817, U30 PC817, U31 PC817, U32 PC817, U33 PC817, U34 PC817, U35 PC817, U36 PC817, U37 PC817, U38 PC817, U39 PC817, U4 JTD1524D05, U40 PC817, U41 PC817, U42 PC817, U43 PC817, U44 PC817, U45 PC817, U46 PC817, U47 PC817, U48 PC817, U5 PC817, U6 PC817, U8 PC817, U9 PC817

Commit message: little fix / adding images
Connections:
- R17 pad 1: gnd -> 3v3
- R18 pad 1: gnd -> 3v3
- R19 pad 1: gnd -> 3v3
- R20 pad 1: gnd -> 3v3
- R21 pad 1: gnd -> 3v3
- R22 pad 1: gnd -> 3v3
- R23 pad 1: gnd -> 3v3
- R24 pad 1: gnd -> 3v3
- R25 pad 1: gnd -> 3v3
- R27 pad 1: gnd -> 3v3
Routing:
- net 3v3: track 290.6 -> 324.6 mm, vias 5 -> 9
